File: Demonstrator_HardwareDesign/PCB_V1/DesignFiles_KiCad6/EHealth_PCB.kicad_pcb (KiCad board)
At the start: 2 copper layers, 50 x 50 mm, 44 parts, among them J1 Conn_01x06, J2 Conn_01x06, J3-MagneticInterconnect1 Conn_01x08, J4 Conn_01x06, J4-OffTheShelf-Digital1 Conn_02x06_Counter_Clockwise, J5-Power1 Conn_01x03, J5-Power2 Conn_01x03, Q1 PMOS, U1 TCA9548APWR, U2 DEBO DCDC DOWN 4

Commit message: huidige layout
Parts:
- added D: TVS Diode 824012823, Resistor_SMD:R_0805_2012Metric_Pad1.20x1.40mm_HandSolder, F.Cu at (189.2, 89.5)
- added D: TVS Diode 824012823, Resistor_SMD:R_0805_2012Metric_Pad1.20x1.40mm_HandSolder, F.Cu at (196.9, 72.4)
- added D: TVS Diode 824012823, Resistor_SMD:R_0805_2012Metric_Pad1.20x1.40mm_HandSolder, F.Cu at (196.9, 61.7)
- added D3: TVS Diode 824012823, Resistor_SMD:R_0805_2012Metric_Pad1.20x1.40mm_HandSolder, F.Cu at (189.2, 75.0)
- added D4: TVS Diode 824012823, Resistor_SMD:R_0805_2012Metric_Pad1.20x1.40mm_HandSolder, F.Cu at (189.2, 79.0)
- added D6: TVS Diode 824012823, Resistor_SMD:R_0805_2012Metric_Pad1.20x1.40mm_HandSolder, F.Cu at (189.2, 85.5)
- added FB: FerriteBead, Resistor_SMD:R_0805_2012Metric_Pad1.20x1.40mm_HandSolder, F.Cu at (196.9, 70.4)
- added FB: FerriteBead, Resistor_SMD:R_0805_2012Metric_Pad1.20x1.40mm_HandSolder, F.Cu at (187.2, 89.5)
- added FB: FerriteBead, Resistor_SMD:R_0805_2012Metric_Pad1.20x1.40mm_HandSolder, F.Cu at (196.9, 63.9)
- added FB3: FerriteBead, Resistor_SMD:R_0805_2012Metric_Pad1.20x1.40mm_HandSolder, F.Cu at (187.2, 75.0)
- added FB4: FerriteBead, Resistor_SMD:R_0805_2012Metric_Pad1.20x1.40mm_HandSolder, F.Cu at (187.2, 79.0)
- added FB6: FerriteBead, Resistor_SMD:R_0805_2012Metric_Pad1.20x1.40mm_HandSolder, F.Cu at (187.2, 85.5)
- added J3: Conn_01x06, Connector_PinHeader_2.54mm:PinHeader_1x08_P2.54mm_Vertical, F.Cu at (197.2, 58.8)
- J2: footprint Connector_PinHeader_2.54mm:PinHeader_1x16_P2.54mm_Vertical -> Connector_PinHeader_2.54mm:PinHeader_1x08_P2.54mm_Vertical
- moved R12 27.0 mm to (191.2, 85.5), turned to -90 degrees
- moved R 25.2 mm to (191.2, 89.5)
- moved R10 23.9 mm to (225.0, 76.4), turned to 180 degrees
- moved R 23.5 mm to (196.9, 66.2), turned to 0 degrees
- moved R 23.3 mm to (196.9, 68.4), turned to 0 degrees
- moved R9 22.6 mm to (225.0, 74.4), turned to 180 degrees
- moved J2 21.3 mm to (209.5, 58.7)
- moved C2 19.5 mm to (223.2, 59.9)
- moved R7 18.8 mm to (191.2, 79.0), turned to 90 degrees
- moved R8 18.4 mm to (191.2, 75.0)
- moved Q 17.0 mm to (206.0, 93.0), turned to 0 degrees
- moved Power 15.4 mm to (215.1, 59.3), turned to 90 degrees
- moved C1 15.1 mm to (212.2, 60.3), turned to 90 degrees
- moved R25 8.41 mm to (226.0, 70.5), turned to -90 degrees
- moved R24 8.26 mm to (223.8, 70.5), turned to -90 degrees
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- renumbered F1 to Fuse, J3-MagneticInterconnect1 to MagneticInterconnect, J5-Power2 to Power, J5-Power1 to Power, Q1 to Q, R3 to R, R2 to R, R6 to R, R11 to R, U1 to U
Connections:
- J2 pad 2: +3.3V -> GND
- J2 pad 3: GND -> Net-(J2-Pin_3)
- J2 pad 4: GND -> Net-(J2-Pin_4)
- J2 pad 5: Net-(J2-Pin_5) -> +3.3V
- J2 pad 6: Net-(J2-Pin_6) -> GND
- J4 pad 13: Net-(J4-Pin_13) -> Net-(D6-A2)
- J4 pad 15: Net-(J4-Pin_15) -> Net-(D5-A2)
- J4 pad 5: Net-(J4-Pin_5) -> Net-(D3-A2)
- J4 pad 7: Net-(J4-Pin_7) -> Net-(D4-A2)
- LOLIN_C3_PICO1 pad 10: Net-(J1-Pin_8) -> Net-(J1-Pin_2)
- LOLIN_C3_PICO1 pad 11: Net-(J1-Pin_6) -> Net-(J1-Pin_4)
- LOLIN_C3_PICO1 pad 12: Net-(J1-Pin_4) -> Net-(J1-Pin_6)
- LOLIN_C3_PICO1 pad 13: Net-(J1-Pin_2) -> Net-(J1-Pin_8)
- MagneticInterconnect pad 3: /SDA -> Net-(D2-A2)
- MagneticInterconnect pad 4: /SCL -> Net-(D1-A2)
- R pad 2: Net-(J4-Pin_15) -> Net-(D5-A2)
- R12 pad 2: Net-(J4-Pin_13) -> Net-(D6-A2)
- R20 pad 2: Net-(J2-Pin_16) -> Net-(J3-Pin_7)
- R21 pad 2: Net-(J2-Pin_14) -> Net-(J3-Pin_8)
- R22 pad 2: Net-(J2-Pin_15) -> Net-(J3-Pin_3)
- R23 pad 2: Net-(J2-Pin_13) -> Net-(J3-Pin_4)
- R24 pad 2: Net-(J2-Pin_8) -> Net-(J2-Pin_7)
- R25 pad 2: Net-(J2-Pin_6) -> Net-(J2-Pin_8)
- R26 pad 2: Net-(J2-Pin_7) -> Net-(J2-Pin_3)
- R27 pad 2: Net-(J2-Pin_5) -> Net-(J2-Pin_4)
- R7 pad 2: Net-(J4-Pin_7) -> Net-(D4-A2)
- R8 pad 2: Net-(J4-Pin_5) -> Net-(D3-A2)
- U pad 13: Net-(J2-Pin_7) -> Net-(J2-Pin_8)
- U pad 14: Net-(J2-Pin_5) -> Net-(J2-Pin_7)
- U pad 15: Net-(J2-Pin_8) -> Net-(J2-Pin_4)
- U pad 16: Net-(J2-Pin_6) -> Net-(J2-Pin_3)
- U pad 17: Net-(J2-Pin_15) -> Net-(J3-Pin_8)
- U pad 18: Net-(J2-Pin_13) -> Net-(J3-Pin_7)
- U pad 19: Net-(J2-Pin_16) -> Net-(J3-Pin_4)
- U pad 20: Net-(J2-Pin_14) -> Net-(J3-Pin_3)
- U pad 4: Net-(J4-Pin_7) -> Net-(U1-SD0)
- U pad 5: Net-(J4-Pin_5) -> Net-(U1-SC0)
- U pad 8: Net-(J4-Pin_15) -> Net-(U1-SD2)
- U pad 9: Net-(J4-Pin_13) -> Net-(U1-SC2)
Routing:
- net +3.3V: track 13.8 -> 305.5 mm, vias 1 -> 18
- net VDD: track 2.70 -> 100.6 mm, vias 0 -> 1
- net GND_12V: track 0.00 -> 72.7 mm, vias 0 -> 1
- net /SDA: track 0.00 -> 59.4 mm, vias 0 -> 3
- net /SCL: track 0.00 -> 58.2 mm, vias 0 -> 4
- net VDD_12V: track 0.00 -> 57.2 mm
- net /SPI_CS: track 0.00 -> 54.1 mm, vias 0 -> 1
- net /A5: track 0.00 -> 53.3 mm, vias 0 -> 2
- net Net-(J2-Pin_8): track 0.00 -> 48.8 mm, vias 0 -> 1
- net Net-(J4-Pin_8): track 0.00 -> 48.5 mm, vias 0 -> 1
- net /GPIO4_LED: track 0.00 -> 47.3 mm, vias 0 -> 1
- net Net-(U1-SC0): track 0.00 -> 46.3 mm, vias 0 -> 2
- net Net-(J4-Pin_16): track 0.00 -> 45.8 mm, vias 0 -> 1
- net Net-(J4-Pin_6): track 0.00 -> 45.8 mm, vias 0 -> 1
- net Net-(J4-Pin_14): track 0.45 -> 45.9 mm, vias 0 -> 3
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Other:
- outline, holes or cut-outs redrawn
- board text added: "3.3V GND SCL SDA"
- board text added: "3.3V GND SDA SCL"
- board text added: "A5"
- board text added: "ANALOG SENSORS"
- board text added: "CS"
- board text added: "EMC protection for long distance communication on row1"
- board text added: "Extra off the shelf sensor pins"
- board text added: "FBEAD DIODE RESISTOR"
- board text added: "LED"
- board text added: "Multiplexer"
- board text added: "Off the shelf sensor pins"
- board text added: "Pull up Multiplexer"
- board text added: "Pull-up Resistors channels"
- board text added: "RST"
- board text added: "RX"
- board text added: "Row1 Row2"
- board text added: "SCL"
- board text added: "SCL line"
- board text added: "SDA"
- board text added: "SDA SCL GND 3.3V"
- board text added: "SDA line"
- board text added: "VDD 3.3V GND"
- board text added: "VDD GND SDA SCL"
- board text added: "reversed polarity protection"
- board text removed: "Analog sensors"
- board text removed: "Antenna position"
- board text removed: "USB connector -->"

Commit message: huidige layout
Parts:
- removed Q: PMOS, Package_SO:Infineon_PG-DSO-8-27_3.9x4.9mm_EP2.65x3mm
- added T: BSC320N20NS3_G, Library-TRANS:PG-TDSON-8, F.Cu at (206.1, 92.9)
- D1, D2, D5: renamed from D; footprint Resistor_SMD:R_0805_2012Metric_Pad1.20x1.40mm_HandSolder -> Resistor_SMD:R_0603_1608Metric_Pad0.98x0.95mm_HandSolder
- D3, D4, D6: footprint Resistor_SMD:R_0805_2012Metric_Pad1.20x1.40mm_HandSolder -> Resistor_SMD:R_0603_1608Metric_Pad0.98x0.95mm_HandSolder
- renumbered C4 to C1, C2 to C1, C5 to C1, C3 to C2, Fuse to F, FB to FB5, R to R11, U to U1
Routing:
- net Net-(T1-D): track 0.00 -> 7.35 mm
- net Net-(T1-S): track 28.7 -> 35.5 mm, vias 1 -> 3
- net Net-(T1-G): track 0.00 -> 3.97 mm
Other:
- outline, holes or cut-outs redrawn
- board text added: "D"
- board text added: "FB"
- board text added: "GPI0 GND"
- board text added: "Pull up"
- board text added: "R"
- board text added: "Row1"
- board text added: "Row2"
- board text added: "SCL SDA GND VDD"
- board text added: "long distance com on row1"
- board text added: "off the shelf sensor pins"
- board text removed: "EMC protection for long distance communication on row1"
- board text removed: "Extra off the shelf sensor pins"
- board text removed: "FBEAD DIODE RESISTOR"
- board text removed: "Pull-up Resistors channels"
- board text removed: "Row1 Row2"
- board text removed: "SDA SCL GND 3.3V"
- board text removed: "VDD GND SDA SCL"
