File: Demonstrator_HardwareDesign/PCB_V1/DesignFiles_KiCad6/EHealth_PCB.kicad_pcb (KiCad board)
At the start: 2 copper layers, 50 x 50 mm, 57 parts, among them J1 Conn_01x06, J2 Conn_01x06, J3 Conn_01x06, J4 Conn_01x06, J4-OffTheShelf-Digital1 Conn_02x06_Counter_Clockwise, U1 TCA9548APWR, U2 DEBO DCDC DOWN 4

Commit message: huidige layout
Routing:
- net +3.3V: track 305.8 -> 307.6 mm
Changed lines of the file:
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@@
 		(tags "resistor handsolder")
 		(property "Reference" "FB"
-			(at -2.873051 0.105157 270)
+			(at -2.873051 0.105157 -90)
 			(layer "F.SilkS")
 			(effects
@@
 			(font
 				(size 0.8 0.8)
-				(thickness 0.16)
+				(thickness 0.15)
 				(bold yes)
 			)
@@
 	)
 	(gr_text "Off the shelf \nsensor pins"
-		(at 186.833811 72.553961 0)
+		(at 186.781284 72.55683 0)
 		(layer "F.SilkS")
 		(effects
@@
 	)
 	(segment
-		(start 205.4 78.8)
-		(end 205.8 79.2)
-		(width 0.25)
-		(layer "F.Cu")
-		(net 3)
-	)
-	(segment
 		(start 223.75 67.885502)
 		(end 223.437098 67.5726)
@@
 	)
 	(segment
-		(start 205.8 79.2)
-		(end 211.306381 79.2)
-		(width 0.25)
-		(layer "F.Cu")
-		(net 3)
-	)
-	(segment
 		(start 204 86)
 		(end 206 86)
@@
 	)
 	(segment
-		(start 203.8 78.2)
-		(end 204.4 78.8)
-		(width 0.25)
-		(layer "F.Cu")
-		(net 3)
-	)
-	(segment
 		(start 181.915724 71.84)
 		(end 184.455724 71.84)
@@
 	)
 	(segment
+		(start 204.8 78.2)
+		(end 205.8 79.2)
+		(width 0.25)
+		(layer "F.Cu")
+		(net 3)
+	)
+	(segment
 		(start 216.9822 68)
 		(end 217.5 68)
@@
 	)
 	(segment
-		(start 212.25 68)
-		(end 212.25 69.25)
+		(start 211.394659 79.111722)
+		(end 211.394659 76.861722)
 		(width 0.25)
 		(layer "F.Cu")
@@
 	)
 	(segment
-		(start 204.218572 58.75)
-		(end 204.218572 57.654028)
+		(start 212.25 68)
+		(end 212.25 69.25)
 		(width 0.25)
 		(layer "F.Cu")
@@
 	)
 	(segment
-		(start 211.306381 79.2)
-		(end 211.394659 79.111722)
+		(start 204.218572 58.75)
+		(end 204.218572 57.654028)
 		(width 0.25)
 		(layer "F.Cu")
@@
 	)
 	(segment
+		(start 205.8 79.2)
+		(end 211.306381 79.2)
+		(width 0.25)
+		(layer "F.Cu")
+		(net 3)
+	)
+	(segment
 		(start 213.686458 102.603958)
 		(end 211.57 100.4875)
@@
 	)
 	(segment
+		(start 203.5 78.2)
+		(end 204.8 78.2)
+		(width 0.25)
+		(layer "F.Cu")
+		(net 3)
+	)
+	(segment
 		(start 224.75 67.5)
 		(end 224.25 68)
@@
 	)
 	(segment
+		(start 211.306381 79.2)
+		(end 211.394659 79.111722)
+		(width 0.25)
+		(layer "F.Cu")
+		(net 3)
+	)
+	(segment
 		(start 223.32 91)
 		(end 219.060449 91)
@@
 	)
 	(segment
-		(start 211.394659 79.111722)
-		(end 211.394659 76.861722)
-		(width 0.25)
-		(layer "F.Cu")
-		(net 3)
-	)
-	(segment
 		(start 181.915724 82)
 		(end 182.335724 82.42)
@@
 	)
 	(segment
-		(start 204.4 78.8)
-		(end 205.4 78.8)
-		(width 0.25)
-		(layer "F.Cu")
-		(net 3)
-	)
-	(segment
 		(start 194.589361 89.291487)
 		(end 198.630848 85.25)
@@
 	)
 	(via
-		(at 203.8 78.2)
+		(at 203.6774 78.2)
 		(size 0.8)
 		(drill 0.4)
@@
 	)
 	(segment
+		(start 203.6774 78.0226)
+		(end 203.6774 77.5226)
+		(width 0.25)
+		(layer "B.Cu")
+		(net 3)
+	)
+	(segment
 		(start 191.25 82.5)
 		(end 191 82.25)
@@
 	)
 	(segment
-		(start 203.8 86.2)
-		(end 203.8 78.2)
+		(start 188.1976 70.75)
+		(end 185.545724 70.75)
 		(width 0.25)
 		(layer "B.Cu")
@@
 	)
 	(segment
-		(start 188.1976 70.75)
-		(end 185.545724 70.75)
+		(start 202 84.4)
+		(end 202 79.7)
 		(width 0.25)
 		(layer "B.Cu")
@@
 	)
 	(segment
+		(start 205.2 76)
+		(end 205.2 74.8)
+		(width 0.25)
+		(layer "B.Cu")
+		(net 3)
+	)
+	(segment
+		(start 203.8 86.2)
+		(end 202 84.4)
+		(width 0.25)
+		(layer "B.Cu")
+		(net 3)
+	)
+	(segment
 		(start 196.8 60)
 		(end 196.2 60.6)
@@
 	)
 	(segment
+		(start 202 79.7)
+		(end 203.6774 78.0226)
+		(width 0.25)
+		(layer "B.Cu")
+		(net 3)
+	)
+	(segment
 		(start 208.27 58.741484)
 		(end 210.058516 58.741484)
@@
 	)
 	(segment
+		(start 203.6774 77.5226)
+		(end 205.2 76)
+		(width 0.25)
+		(layer "B.Cu")
+		(net 3)
+	)
+	(segment
 		(start 224.6 86.2)
 		(end 224.65 86.15)
@@
 	)
 	(segment
-		(start 205.2 76.8)
-		(end 203.8 78.2)
-		(width 0.25)
-		(layer "B.Cu")
-		(net 3)
-	)
-	(segment
 		(start 191.25 82)
 		(end 191 82.25)
@@
 	)
 	(segment
-		(start 208.2 71.8)
-		(end 205.2 74.8)
-		(width 0.25)
-		(layer "B.Cu")
-		(net 3)
-	)
-	(segment
 		(start 209.5178 68.25)
 		(end 209.5 68.2322)
@@
 	)
 	(segment
-		(start 205.2 74.8)
-		(end 205.2 76.8)
+		(start 192.558863 89.411344)
+		(end 192.67872 89.291487)
 		(width 0.25)
 		(layer "B.Cu")
@@
 	)
 	(segment
-		(start 192.558863 89.411344)
-		(end 192.67872 89.291487)
+		(start 192.15 60.6)
+		(end 191.75 61)
 		(width 0.25)
 		(layer "B.Cu")
@@
 	)
 	(segment
-		(start 192.15 60.6)
-		(end 191.75 61)
+		(start 205.2 74.8)
+		(end 208.2 71.8)
 		(width 0.25)
 		(layer "B.Cu")
@@
 	)
 	(segment
-		(start 218.2226 85.5)
-		(end 220.5 85.5)
-		(width 0.25)
-		(layer "F.Cu")
-		(net 15)
-	)
-	(segment
-		(start 223.2 88.2)
-		(end 223.58 88.2)
+		(start 195.64168 79.8226)
+		(end 192.9024 77.08332)
 		(width 0.25)
 		(layer "F.Cu")
@@
 	)
 	(segment
-		(start 183.92 68.75)
-		(end 181.92 66.75)
+		(start 218.2226 85.5)
+		(end 220.5 85.5)
 		(width 0.25)
 		(layer "F.Cu")
@@
 	)
 	(segment
-		(start 205 79.8)
-		(end 205.022593 79.822593)
+		(start 223.2 88.2)
+		(end 223.58 88.2)
 		(width 0.25)
 		(layer "F.Cu")
@@
 	)
 	(segment
-		(start 195.64168 79.8226)
-		(end 192.9024 77.08332)
+		(start 220.5 85.5)
+		(end 223.2 88.2)
 		(width 0.25)
 		(layer "F.Cu")
@@
 	)
 	(segment
-		(start 220.5 85.5)
-		(end 223.2 88.2)
-		(width 0.25)
-		(layer "F.Cu")
-		(net 15)
-	)
-	(segment
 		(start 192.9024 77.08332)
 		(end 192.9024 73.42872)
@@
 	)
 	(segment
-		(start 205.022586 79.8226)
+		(start 203.6774 79.8226)
 		(end 195.64168 79.8226)
 		(width 0.25)
@@
 	)
 	(segment
-		(start 205.022593 79.822593)
-		(end 205.022586 79.8226)
+		(start 183.92 68.75)
+		(end 181.92 66.75)
 		(width 0.25)
 		(layer "F.Cu")
@@
 	)
 	(via
-		(at 205 79.8)
+		(at 203.6774 79.8226)
 		(size 0.8)
 		(drill 0.4)
@@
 	)
 	(segment
-		(start 211.6 85.8)
-		(end 217.9226 85.8)
+		(start 205.6226 79.8226)
+		(end 211.6 85.8)
 		(width 0.25)
 		(layer "B.Cu")
@@
 	)
 	(segment
-		(start 217.9226 85.8)
-		(end 218 85.7226)
+		(start 211.6 85.8)
+		(end 217.9226 85.8)
 		(width 0.25)
 		(layer "B.Cu")
@@
 	)
 	(segment
-		(start 205.6 79.8)
-		(end 211.6 85.8)
+		(start 217.9226 85.8)
+		(end 218 85.7226)
 		(width 0.25)
 		(layer "B.Cu")
@@
 	)
 	(segment
-		(start 205 79.8)
-		(end 205.6 79.8)
+		(start 203.6774 79.8226)
+		(end 205.6226 79.8226)
 		(width 0.25)
 		(layer "B.Cu")

Commit message: finished layout met logo
Parts:
- added G***: LOGO, LOGO, B.Cu at (218.6, 74.7)
