File: Demonstrator_HardwareDesign/PCB_V1/DesignFiles_KiCad6/EHealth_PCB.kicad_sch (KiCad schematic)
At the start: 57 parts, among them J1 Conn_01x06, J2 Conn_01x06, J3 Conn_01x06, J3-MagneticInterconnect1 Conn_01x08, J4 Conn_01x06, J4-OffTheShelf-Digital1 Conn_02x06_Counter_Clockwise, J5-Power1 Conn_01x03, J5-Power2 Conn_01x03, Q1 PMOS, U1 TCA9548APWR, U2 DEBO DCDC DOWN 4

Commit message: huidige layout
Parts:
- removed Q1: PMOS, Library-TRANS:PG-TDSON-8, symbol Simulation_SPICE:PMOS
- added T1: BSC320N20NS3_G, Library-TRANS:PG-TDSON-8, symbol Infineon:BSC320N20NS3_G
Connections:
- net at R6.1: now also T1.4 (G)
- net at U2.2 (+Vin): now also T1.1 (S)
- net at F1.2: now also T1.5 (D)
Changed lines of the file:
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@@
 	(wire
 		(pts
-			(xy 67.31 132.08) (xy 68.58 132.08)
+			(xy 67.31 132.08) (xy 71.12 132.08)
 		)
 		(stroke
@@
 	(wire
 		(pts
-			(xy 78.74 132.08) (xy 88.9 132.08)
+			(xy 76.2 132.08) (xy 88.9 132.08)
 		)
 		(stroke
@@
 	(wire
 		(pts
-			(xy 73.66 139.7) (xy 73.66 152.4)
+			(xy 73.66 134.62) (xy 73.66 152.4)
 		)
 		(stroke
@@
 	)
 	(symbol
-		(lib_id "Simulation_SPICE:PMOS")
-		(at 73.66 134.62 90)
-		(unit 1)
-		(exclude_from_sim no)
-		(in_bom yes)
-		(on_board yes)
-		(dnp no)
-		(fields_autoplaced yes)
-		(property "Reference" "Q1"
-			(at 73.66 125.73 90)
-			(effects
-				(font
-					(size 1.27 1.27)
-				)
-			)
-		)
-		(property "Value" "PMOS"
-			(at 73.66 128.27 90)
-			(effects
-				(font
-					(size 1.27 1.27)
-				)
-			)
-		)
-		(property "Footprint" "Library-TRANS:PG-TDSON-8"
-			(at 71.12 129.54 0)
-			(effects
-				(font
-					(size 1.27 1.27)
-				)
-				(hide yes)
-			)
-		)
-		(property "Datasheet" "https://ngspice.sourceforge.io/docs/ngspice-html-manual/manual.xhtml#cha_MOSFETs"
-			(at 86.36 134.62 0)
-			(effects
-				(font
-					(size 1.27 1.27)
-				)
-				(hide yes)
-			)
-		)
-		(property "Description" "P-MOSFET transistor, drain/source/gate"
-			(at 73.66 134.62 0)
-			(effects
-				(font
-					(size 1.27 1.27)
-				)
-				(hide yes)
-			)
-		)
-		(property "Sim.Device" "PMOS"
-			(at 90.805 134.62 0)
-			(effects
-				(font
-					(size 1.27 1.27)
-				)
-				(hide yes)
-			)
-		)
-		(property "Sim.Type" "VDMOS"
-			(at 92.71 134.62 0)
-			(effects
-				(font
-					(size 1.27 1.27)
-				)
-				(hide yes)
-			)
-		)
-		(property "Sim.Pins" "1=D 2=G 3=S"
-			(at 88.9 134.62 0)
-			(effects
-				(font
-					(size 1.27 1.27)
-				)
-				(hide yes)
-			)
-		)
-		(pin "2"
-		)
-		(pin "1"
-		)
-		(pin "3"
-		)
-		(instances
-			(project "EHealth_PCB"
-				(path "/2780e3fe-bae0-409b-b243-5af753ed0cfc"
-					(reference "Q1")
-					(unit 1)
-				)
-			)
-		)
-	)
-	(symbol
 		(lib_id "Device:C_Small")
 		(at 256.54 49.53 0)
@@
 					(unit 1)
 				)
+			)
+		)
+	)
+	(symbol
+		(lib_id "Infineon:BSC320N20NS3_G")
+		(at 73.66 132.08 90)
+		(unit 1)
+		(exclude_from_sim no)
+		(in_bom yes)
+		(on_board yes)
+		(dnp no)
+		(fields_autoplaced yes)
+		(property "Reference" "T1"
+			(at 77.47 130.6829 90)
+			(effects
+				(font
+					(size 1.524 1.524)
+				)
+				(justify right)
+			)
+		)
+		(property "Value" "BSC320N20NS3_G"
+			(at 77.47 133.2229 90)
+			(effects
+				(font
+					(size 1.524 1.524)
+				)
+				(justify right)
+			)
+		)
+		(property "Footprint" "Library-TRANS:PG-TDSON-8"
+			(at 68.58 132.08 0)
+			(effects
+				(font
+					(size 1.524 1.524)
+				)
+				(hide yes)
+			)
+		)
+		(property "Datasheet" ""
+			(at 68.58 132.08 0)
+			(effects
+				(font
+					(size 1.524 1.524)
+				)
+				(hide yes)
+			)
+		)
+		(property "Description" "200V 36A 22nC  27m  OptiMOS"
+			(at 68.58 132.08 0)
+			(effects
+				(font
+					(size 1.524 1.524)
+				)
+				(hide yes)
+			)
+		)
+		(property "Voltage" "200V"
+			(at 68.58 134.62 0)
+			(effects
+				(font
+					(size 1.524 1.524)
+				)
+				(hide yes)
+			)
+		)
+		(property "Amps" "36A"
+			(at 68.58 127 0)
+			(effects
+				(font
+					(size 1.524 1.524)
+				)
+				(hide yes)
+			)
+		)
+		(property "Edit" "2017-05-30"
+			(at 68.58 133.35 0)
+			(effects
+				(font
+					(size 1.524 1.524)
+				)
+				(hide yes)
+			)
+		)
+		(property "Qg" "22nC"
+			(at 68.58 137.16 0)
+			(effects
+				(font
+					(size 1.524 1.524)
+				)
+				(hide yes)
+			)
+		)
+		(property "RDS" "27"
+			(at 68.58 133.35 0)
+			(effects
+				(font
+					(size 1.524 1.524)
+				)
+				(hide yes)
+			)
+		)
+		(pin "5"
+		)
+		(pin "4"
+		)
+		(pin "1"
+		)
+		(instances
+			(project "EHealth_PCB"
+				(path "/2780e3fe-bae0-409b-b243-5af753ed0cfc"
+					(reference "T1")
+					(unit 1)
+				)

Commit message: huidige layout
Changed lines of the file:
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@@
-		)
-	)
-	(label "SPI_MISO"
-		(at 34.29 179.07 180)
-		(fields_autoplaced yes)
-		(effects
-			(font
-				(size 1.27 1.27)
-			)
-			(justify right bottom)
 		)
 	)
@@
 					(unit 1)
 				)
-			)
-		)
-	)
-	(symbol
-		(lib_id "power:+3.3V")
-		(at 232.41 62.23 90)
-		(unit 1)
-		(exclude_from_sim no)
-		(in_bom yes)
-		(on_board yes)
-		(dnp no)
-		(property "Reference" "#PWR042"
-			(at 236.22 62.23 0)
-			(effects
-				(font
-					(size 1.27 1.27)
-				)
-				(hide yes)
-			)
-		)
-		(property "Value" "+3.3V"
-			(at 228.6 62.23 90)
-			(effects
-				(font
-					(size 1.27 1.27)
-				)
-				(justify left)
-			)
-		)
-		(property "Footprint" ""
-			(at 232.41 62.23 0)
-			(effects
-				(font
-					(size 1.27 1.27)
-				)
-				(hide yes)
-			)
-		)
-		(property "Datasheet" ""
-			(at 232.41 62.23 0)
-			(effects
-				(font
-					(size 1.27 1.27)
-				)
-				(hide yes)
-			)
-		)
-		(property "Description" ""
-			(at 232.41 62.23 0)
-			(effects
-				(font
-					(size 1.27 1.27)
-				)
-				(hide yes)
-			)
-		)
-		(pin "1"
-		)
-		(instances
-			(project "EHealth_PCB"
-				(path "/2780e3fe-bae0-409b-b243-5af753ed0cfc"
-					(reference "#PWR042")
-					(unit 1)
-				)
