File: Demonstrator_HardwareDesign/PCB_V1/DesignFiles_KiCad6/Hybrid E-tattoo Hub V2_0/EHealth_PCB.kicad_pcb (KiCad board)
At the start: 2 copper layers, 50 x 50 mm, 58 parts, among them J1 Conn_01x06, J2 Conn_01x06, J3 Conn_01x06, J4 Conn_01x06, J4-OffTheShelf-Digital1 Conn_02x06_Counter_Clockwise, U1 TCA9548APWR, U2 DEBO DCDC DOWN 4

Commit message: verbeterde layout
Parts:
- removed R (x3): R, Resistor_SMD:R_0805_2012Metric_Pad1.20x1.40mm_HandSolder
- C3: renamed from C2; value C_Small -> 10uF
- J2: footprint Connector_PinHeader_2.54mm:PinHeader_1x08_P2.54mm_Vertical -> Connector_PinHeader_2.54mm:PinHeader_1x04_P2.54mm_Vertical
- R1, R4, R5: value R -> 1K
- R17: value R -> 220
- R27, R8: value R -> 3.3K
- moved G*** 38.5 mm to (188.8, 99.0)
- moved D1 4.33 mm to (196.9, 66.0)
- moved FB2 4.08 mm to (196.9, 68.0)
- moved J2 1.06 mm to (210.6, 58.8)
- moved FB1 0.40 mm to (196.9, 70.0)
- moved D2 0.36 mm to (196.9, 72.0)
- renumbered C1 to C2, C1 to C4, C1 to C5, F to F1, FB to FB1, FB to FB2, MagneticInterconnect to J3-MagneticInterconnect1, Power to J5-Power1, Power to J5-Power2, T to T1
Connections:
- FB1 pad 1: /SDA -> /SDA_mult
- FB2 pad 2: /SCL -> /SCL_mult
- R24 pad 2: Net-(J2-Pin_7) -> /SCL_mult
- R25 pad 2: Net-(J2-Pin_8) -> /SDA_mult
- T1 pad 4: Net-(T1-G) -> GND_12V
- U1 pad 13: Net-(J2-Pin_8) -> /SDA_mult
- U1 pad 14: Net-(J2-Pin_7) -> /SCL_mult
- U2 pad 1: GND_12V -> Net-(T1-S)
- U2 pad 2: Net-(T1-S) -> GND_12V
- U2 pad 3: GND -> VDD
- U2 pad 4: VDD -> GND
Routing:
- net Net-(J2-Pin_8): track 48.8 -> 0.00 mm, vias 1 -> 0
- net Net-(J2-Pin_7): track 43.9 -> 0.00 mm, vias 1 -> 0
- net /SDA_mult: track 0.00 -> 40.0 mm, vias 0 -> 2
- net /SCL_mult: track 0.00 -> 36.0 mm, vias 0 -> 2
- net +3.3V: track 307.6 -> 292.5 mm, vias 18 -> 16
- net GND_12V: track 72.7 -> 62.6 mm, vias 1 -> 2
- net GND: track 47.6 -> 38.3 mm
- net /SDA: track 59.4 -> 68.4 mm, vias 3 -> 5
- net VDD: track 100.6 -> 92.7 mm, vias 1 -> 0
- net /SCL: track 58.2 -> 64.5 mm, vias 4 -> 3
- net Net-(T1-S): track 35.5 -> 30.8 mm, vias 3 -> 0
- net Net-(T1-G): track 3.97 -> 0.00 mm
- net Net-(D1-A2): track 9.96 -> 13.1 mm
- net Net-(U1-SC0): track 46.3 -> 43.8 mm
- net /GPIO20_RX: track 33.2 -> 35.0 mm
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Other:
- board text removed: "SCL line"
- board text removed: "SDA line"

Commit message: up to date
Parts:
- T1: footprint Library-TRANS:PG-TDSON-8 -> Package_SON:Infineon_PG-TDSON-8_6.15x5.15mm
- moved F1 0.37 mm to (200.8, 89.8)
- turned T1 to 0 degrees
Connections:
- U2 pad 1: Net-(T1-S) -> GND_12V
- U2 pad 2: GND_12V -> Net-(T1-S)
- U2 pad 3: VDD -> GND
- U2 pad 4: GND -> VDD
Routing:
- net GND: track 38.3 -> 34.3 mm
- net Net-(T1-S): track 30.8 -> 28.0 mm
- net /GPIO4_LED: track 49.2 -> 48.0 mm
- net /SPI_CS: track 55.9 -> 55.1 mm
- net /GPIO21_TX: track 27.4 -> 28.0 mm
Other:
- board text removed: "off the shelf sensor pins"

Commit message: PCB up to date
Parts:
- moved F1 14.3 mm to (215.0, 91.2), turned to 180 degrees
- moved D1 3.61 mm to (196.0, 62.5)
- moved D2 3.61 mm to (196.0, 68.5)
- moved FB1 3.61 mm to (196.0, 66.5)
- moved FB2 3.61 mm to (196.0, 64.5)
- moved C3 3.28 mm to (225.0, 84.5), turned to 180 degrees
- moved T1 2.50 mm to (208.6, 92.9)
- moved D3 1.68 mm to (189.5, 73.4)
- moved D4 1.68 mm to (189.6, 77.3)
- moved D5 1.68 mm to (189.6, 87.8)
- moved D6 1.68 mm to (189.6, 83.8)
- moved FB3 1.68 mm to (187.5, 73.4)
- moved FB4 1.68 mm to (187.6, 77.3)
- moved FB5 1.68 mm to (187.6, 87.8)
- moved FB6 1.68 mm to (187.6, 83.8)
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- renumbered J3-MagneticInterconnect1 to MagneticInterconnect, J5-Power2 to Power, J5-Power1 to Power
Routing:
- net VDD_12V: track 57.2 -> 72.3 mm
- net GND_12V: track 62.8 -> 71.0 mm, vias 2 -> 1
- net Net-(T1-S): track 28.0 -> 34.7 mm
- net GND: track 34.3 -> 40.1 mm, vias 12 -> 11
- net Net-(D1-A2): track 13.1 -> 8.37 mm
- net Net-(D2-A2): track 16.9 -> 12.8 mm
- net /SDA_mult: track 40.0 -> 43.3 mm
- net /GPIO21_TX: track 28.0 -> 24.7 mm
- net /GPIO20_RX: track 34.8 -> 32.0 mm
- net /SCL_mult: track 36.0 -> 38.5 mm
- net Net-(T1-D): track 7.35 -> 5.16 mm
- net Net-(U1-SD2): track 44.9 -> 43.0 mm
- net /SPI_CS: track 55.1 -> 53.3 mm
- net /GPIO4_LED: track 48.0 -> 46.2 mm
- net Net-(J4-Pin_6): track 45.8 -> 47.5 mm
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Other:
- outline, holes or cut-outs redrawn
- board text added: "License to Kill - Bob Dylan -"
- board text added: "Multiplexer sensor pins"
- board text removed: "Off the shelf sensor pins"
