File: Demonstrator_HardwareDesign/PCB_V1/DesignFiles_KiCad6/Hybrid E-tattoo Hub V2_0/EHealth_PCB.kicad_sch (KiCad schematic)
At the start: 57 parts, among them J1 Conn_01x06, J2 Conn_01x06, J3 Conn_01x06, J3-MagneticInterconnect1 Conn_01x08, J4 Conn_01x06, J4-OffTheShelf-Digital1 Conn_02x06_Counter_Clockwise, J5-Power1 Conn_01x03, J5-Power2 Conn_01x03, T1 BSC320N20NS3_G, U1 TCA9548APWR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

Commit message: verbeterde layout
Parts:
- removed J2: Conn_01x06, Connector_PinHeader_2.54mm:PinHeader_1x08_P2.54mm_Vertical, symbol Connector_Generic:Conn_01x08
- removed R2, R3, R6: R, Resistor_SMD:R_0805_2012Metric_Pad1.20x1.40mm_HandSolder, symbol Device:R
- added J2: Conn_01x06, Connector_PinHeader_2.54mm:PinHeader_1x04_P2.54mm_Vertical, symbol Connector_Generic:Conn_01x04
- C3: value C_Small -> 10uF
- R1, R4, R5: value R -> 1K
- R17: value R -> 220
- R27, R8: value R -> 3.3K
Connections:
- net +3.3V: now also J2.1 (Pin_1)
- net GND: now also U2.4 (+Vout), J2.2 (Pin_2); no longer U2.3 (-Vout)
- net GND_12V: now also T1.4 (G), U2.2 (+Vin); no longer U2.1 (-Vin)
- net SCL: no longer FB2.2
- net SDA: no longer FB1.1
- net VDD: now also U2.3 (-Vout); no longer U2.4 (+Vout)
- net SCL_mult: now reaches R24.2, U1.14 (SC4)
- net SCL_mult: now also FB2.2
- net at R26.2, U1.16 (SC5): now also J2.3 (Pin_3)
- net at T1.1 (S): now also U2.1 (-Vin); no longer U2.2 (+Vin)
- net at R27.2, U1.15 (SD5): now also J2.4 (Pin_4)
- net SDA_mult: now reaches R25.2, U1.13 (SD4)
- net SDA_mult: now also FB1.1

Commit message: up to date
Parts:
- T1: footprint Library-TRANS:PG-TDSON-8 -> Package_SON:Infineon_PG-TDSON-8_6.15x5.15mm
Connections:
- net GND: now also U2.3 (-Vout); no longer U2.4 (+Vout)
- net GND_12V: now also U2.1 (-Vin); no longer U2.2 (+Vin)
- net VDD: now also U2.4 (+Vout); no longer U2.3 (-Vout)
- net at T1.1 (S): now also U2.2 (+Vin); no longer U2.1 (-Vin)
Other:
- moved on the sheet: U2

Commit message: PCB up to date
Other:
- moved on the sheet: R1, R4
Changed lines of the file:
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@@
 	(wire
 		(pts
-			(xy 102.87 102.87) (xy 102.87 107.95)
+			(xy 102.87 102.87) (xy 102.87 105.41)
 		)
 		(stroke
@@
 	(wire
 		(pts
-			(xy 110.49 123.19) (xy 113.03 123.19)
+			(xy 110.49 120.65) (xy 113.03 120.65)
 		)
 		(stroke
@@
 	(wire
 		(pts
-			(xy 100.33 118.11) (xy 102.87 118.11)
+			(xy 100.33 115.57) (xy 102.87 115.57)
 		)
 		(stroke
@@
 	(wire
 		(pts
-			(xy 110.49 105.41) (xy 110.49 118.11)
+			(xy 110.49 105.41) (xy 110.49 115.57)
 		)
 		(stroke
@@
 	(wire
 		(pts
-			(xy 113.03 105.41) (xy 113.03 123.19)
+			(xy 113.03 105.41) (xy 113.03 120.65)
 		)
 		(stroke
@@
 	(wire
 		(pts
-			(xy 100.33 123.19) (xy 102.87 123.19)
+			(xy 100.33 120.65) (xy 102.87 120.65)
 		)
 		(stroke
@@
 	(symbol
 		(lib_id "power:GND")
-		(at 102.87 107.95 0)
+		(at 102.87 105.41 0)
 		(unit 1)
 		(exclude_from_sim no)
@@
 		(fields_autoplaced yes)
 		(property "Reference" "#PWR015"
-			(at 102.87 114.3 0)
+			(at 102.87 111.76 0)
 			(effects
 				(font
@@
 		)
 		(property "Value" "GND"
-			(at 102.87 111.76 90)
+			(at 102.87 109.22 90)
 			(effects
 				(font
@@
 		)
 		(property "Footprint" ""
-			(at 102.87 107.95 0)
+			(at 102.87 105.41 0)
 			(effects
 				(font
@@
 		)
 		(property "Datasheet" ""
-			(at 102.87 107.95 0)
+			(at 102.87 105.41 0)
 			(effects
 				(font
@@
 		)
 		(property "Description" ""
-			(at 102.87 107.95 0)
+			(at 102.87 105.41 0)
 			(effects
 				(font
@@
 	(symbol
 		(lib_id "Device:R")
-		(at 106.68 123.19 90)
+		(at 106.68 120.65 90)
 		(unit 1)
 		(exclude_from_sim no)
@@
 		(dnp no)
 		(property "Reference" "R4"
-			(at 107.95 125.73 90)
+			(at 107.95 123.19 90)
 			(effects
 				(font
@@
 		)
 		(property "Value" "1K"
-			(at 104.14 125.73 90)
+			(at 104.14 123.19 90)
 			(effects
 				(font
@@
 		)
 		(property "Footprint" "Resistor_SMD:R_0805_2012Metric_Pad1.20x1.40mm_HandSolder"
-			(at 106.68 124.968 90)
+			(at 106.68 122.428 90)
 			(effects
 				(font
@@
 		)
 		(property "Datasheet" "~"
-			(at 106.68 123.19 0)
+			(at 106.68 120.65 0)
 			(effects
 				(font
@@
 		)
 		(property "Description" ""
-			(at 106.68 123.19 0)
+			(at 106.68 120.65 0)
 			(effects
 				(font
@@
 	(symbol
 		(lib_id "power:+3.3V")
-		(at 100.33 118.11 90)
+		(at 100.33 115.57 90)
 		(unit 1)
 		(exclude_from_sim no)
@@
 		(dnp no)
 		(property "Reference" "#PWR016"
-			(at 104.14 118.11 0)
+			(at 104.14 115.57 0)
 			(effects
 				(font
@@
 		)
 		(property "Value" "+3.3V"
-			(at 96.52 118.11 90)
+			(at 96.52 115.57 90)
 			(effects
 				(font
@@
 		)
 		(property "Footprint" ""
-			(at 100.33 118.11 0)
+			(at 100.33 115.57 0)
 			(effects
 				(font
@@
 		)
 		(property "Datasheet" ""
-			(at 100.33 118.11 0)
+			(at 100.33 115.57 0)
 			(effects
 				(font
@@
 		)
 		(property "Description" ""
-			(at 100.33 118.11 0)
+			(at 100.33 115.57 0)
 			(effects
 				(font
@@
 	(symbol
 		(lib_id "Device:R")
-		(at 106.68 118.11 90)
+		(at 106.68 115.57 90)
 		(unit 1)
 		(exclude_from_sim no)
@@
 		(dnp no)
 		(property "Reference" "R1"
-			(at 107.95 120.65 90)
+			(at 107.95 118.11 90)
 			(effects
 				(font
@@
 		)
 		(property "Value" "1K"
-			(at 104.14 120.65 90)
+			(at 104.14 118.11 90)
 			(effects
 				(font
@@
 		)
 		(property "Footprint" "Resistor_SMD:R_0805_2012Metric_Pad1.20x1.40mm_HandSolder"
-			(at 106.68 119.888 90)
+			(at 106.68 117.348 90)
 			(effects
 				(font
@@
 		)
 		(property "Datasheet" "~"
-			(at 106.68 118.11 0)
+			(at 106.68 115.57 0)
 			(effects
 				(font
@@
 		)
 		(property "Description" ""
-			(at 106.68 118.11 0)
+			(at 106.68 115.57 0)
 			(effects
 				(font
@@
 	(symbol
 		(lib_id "power:+3.3V")
-		(at 100.33 123.19 90)
+		(at 100.33 120.65 90)
 		(unit 1)
 		(exclude_from_sim no)
@@
 		(dnp no)
 		(property "Reference" "#PWR019"
-			(at 104.14 123.19 0)
+			(at 104.14 120.65 0)
 			(effects
 				(font
@@
 		)
 		(property "Value" "+3.3V"
-			(at 96.52 123.19 90)
+			(at 96.52 120.65 90)
 			(effects
 				(font
@@
 		)
 		(property "Footprint" ""
-			(at 100.33 123.19 0)
+			(at 100.33 120.65 0)
 			(effects
 				(font
@@
 		)
 		(property "Datasheet" ""
-			(at 100.33 123.19 0)
+			(at 100.33 120.65 0)
 			(effects
 				(font
@@
 		)
 		(property "Description" ""
-			(at 100.33 123.19 0)
+			(at 100.33 120.65 0)
 			(effects
 				(font
@@
 		(dnp no)
 		(property "Reference" "J4"
-			(at 17.018 85.598 0)
+			(at 26.67 100.838 0)
 			(effects
 				(font
@@
 		)
 		(property "Value" "Conn_01x06"
-			(at 17.78 89.916 0)
+			(at 26.67 103.632 0)
 			(effects
 				(font
